File: PCBs/DC-DC Board/DC-DC Board.kicad_pcb (KiCad board)
At the start: 2 copper layers, 58.4 x 36.8 mm, 38 parts, among them J1 Conn_01x01, J2 Conn_01x01, J3 Conn_01x01, J4 Conn_01x01, J5 Conn_01x02, J6 Conn_01x02, Q1 Q_NMOS_GDS, U1 DBQ0135V2, U2 ACS711, U3 NCP551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

Commit message: Gerber Generation
Oops should not have done this in the actuator branch but here we are loll. Just exported the gerber files for the DCDC / DCDC Micro & the PD Board. Should not affect what you guys are doing.
Other:
- rule trace_min: 0.25 -> 0.2
Changed lines of the file:
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@@
     (zone_clearance 0.25)
     (zone_45_only no)
-    (trace_min 0.25)
+    (trace_min 0.2)
     (segment_width 0.2)
     (edge_width 0.15)
@@
     (visible_elements 7FFFF7FF)
     (pcbplotparams
-      (layerselection 0x010fc_ffffffff)
-      (usegerberextensions false)
+      (layerselection 0x010f0_ffffffff)
+      (usegerberextensions true)
       (usegerberattributes false)
       (usegerberadvancedattributes false)
@@
       (padsonsilk false)
       (subtractmaskfromsilk false)
-      (outputformat 4)
-      (mirror true)
+      (outputformat 1)
+      (mirror false)
       (drillshape 0)
       (scaleselection 1)
-      (outputdirectory ""))
+      (outputdirectory "Gerbers/"))
   )
   (net 0 "")
@@
   (gr_line (start 129.2 33.585) (end 129.2 66.415) (layer Edge.Cuts) (width 0.15))
   (gr_line (start 72.8 31.585) (end 127.2 31.585) (layer Edge.Cuts) (width 0.15))
-  (via (at 122 51.725) (size 0.8) (drill 0.4) (layers F.Cu B.Cu) (net 3))
   (via (at 81.1 58.2) (size 0.6) (drill 0.3) (layers F.Cu B.Cu) (net 1))
   (via (at 82.7 57.3) (size 0.6) (drill 0.3) (layers F.Cu B.Cu) (net 1))
@@
   (via (at 122.5 56.34) (size 0.8) (drill 0.4) (layers F.Cu B.Cu) (net 2))
   (via (at 127.49 64.52) (size 0.8) (drill 0.4) (layers F.Cu B.Cu) (net 2))
+  (via (at 122 51.725) (size 0.8) (drill 0.4) (layers F.Cu B.Cu) (net 3))
   (segment (start 124.87 42.38) (end 125.4 42.38) (width 0.25) (layer F.Cu) (net 3))
   (via (at 98.05 57.9) (size 0.8) (drill 0.4) (layers F.Cu B.Cu) (net 3))
@@
     (polygon
       (pts
-        (xy 80.227121 58.25) (xy 80.227121 56.1) (xy 72.977121 56.05) (xy 73.027121 59.1) (xy 80.227121 59.1)
+        (xy 80.227121 58.25) (xy 80.227121 56.1) (xy 70.32 56.04) (xy 70.37 59.09) (xy 80.227121 59.1)
         (xy 80.227121 58.75)
       )
@@
     (polygon
       (pts
-        (xy 80.229927 58.24262) (xy 80.229927 56.09262) (xy 72.979927 56.04262) (xy 73.029927 59.09262) (xy 80.229927 59.09262)
+        (xy 80.229927 58.24262) (xy 80.229927 56.09262) (xy 70.33 56.03) (xy 70.38 59.08) (xy 80.229927 59.09262)
         (xy 80.229927 58.74262)
       )
