File: PCBs/Tooling Board/DCMotor5-6.sch (KiCad schematic (older format))
At the start: 10 parts

Commit message: Added Sensors
-Added pH Circuit and spec'd components
-Added Pressure sensor connecter
-Added External Temp sensor connector
-Added metal detector connector + input circuit

Need to add IMU interface now (not hard)
Parts:
- removed C? (x2): 100nF, symbol Device:C
- removed J?: Screw Terminal, symbol Connector:Screw_Terminal_01x01
- removed R?: 0.5, symbol Device:R_US
- removed U?: LN298P, symbol EER:LN298P
- removed U?: 74LVC2G14, symbol EER:74LVC2G14
- added C? (x2): 100nF, symbol Device:C
- added J?: Screw Terminal, symbol Connector:Screw_Terminal_01x01
- added R?: 0.5, symbol Device:R_US
- added U?: LN298P, symbol EER:LN298P
- added U?: 74LVC2G14, symbol EER:74LVC2G14
Changed lines of the file:
@@
 $Descr A4 11693 8268
 encoding utf-8
-Sheet 6 7
+Sheet 6 8
 Title ""
 Date ""
@@
 $Comp
 L EER:LN298P U?
-U 1 1 5C4C7247
+U 1 1 5C4E06F9
 P 5730 3140
 F 0 "U?" H 5730 4305 50  0000 C CNN
@@
 $Comp
 L Connector:Screw_Terminal_01x01 J?
-U 1 1 5C4C7477
+U 1 1 5C4E06FB
 P 8200 2840
 F 0 "J?" H 8279 2882 50  0000 L CNN
@@
 $Comp
 L power:GND #PWR?
-U 1 1 5C4C7BF9
+U 1 1 5C4E0703
 P 6980 2590
 F 0 "#PWR?" H 6980 2340 50  0001 C CNN
@@
 $Comp
 L power:GND #PWR?
-U 1 1 5C4C7C15
+U 1 1 5C4E0704
 P 4500 2600
 F 0 "#PWR?" H 4500 2350 50  0001 C CNN
@@
 $Comp
 L power:GND #PWR?
-U 1 1 5C4C7C2A
+U 1 1 5C4E0707
 P 4660 4370
 F 0 "#PWR?" H 4660 4120 50  0001 C CNN
@@
 $Comp
 L power:GND #PWR?
-U 1 1 5C4C7C7B
+U 1 1 5C4E0708
 P 6950 4300
 F 0 "#PWR?" H 6950 4050 50  0001 C CNN
@@
 $Comp
 L Device:C C?
-U 1 1 5C4C8744
+U 1 1 5C4E070B
 P 3980 3490
 F 0 "C?" H 4095 3536 50  0000 L CNN
@@
 $Comp
 L Device:C C?
-U 1 1 5C4C9D1A
+U 1 1 5C4E070E
 P 7320 4150
 F 0 "C?" H 7435 4196 50  0000 L CNN
@@
 $Comp
 L power:GND #PWR?
-U 1 1 5C4C9D20
+U 1 1 5C4E0710
 P 7320 4450
 F 0 "#PWR?" H 7320 4200 50  0001 C CNN
@@
 $Comp
 L power:+5V #PWR?
-U 1 1 5C4C9F8F
+U 1 1 5C4E0712
 P 7320 3760
 F 0 "#PWR?" H 7320 3610 50  0001 C CNN
@@
 $Comp
 L power:+12V #PWR?
-U 1 1 5C4C9FF7
+U 1 1 5C4E0714
 P 4210 3190
 F 0 "#PWR?" H 4210 3040 50  0001 C CNN
@@
 $Comp
 L Device:R_US R?
-U 1 1 5C4CABF0
+U 1 1 5C4E0716
 P 6650 2440
 F 0 "R?" V 6540 2610 50  0000 C CNN
@@
 $Comp
 L EER:74LVC2G14 U?
-U 1 1 5C4CF224
+U 1 1 5C4E071B
 P 2460 5130
 F 0 "U?" H 2460 5645 50  0000 C CNN
@@
 $Comp
 L power:GND #PWR?
-U 1 1 5C4D22A3
+U 1 1 5C4E071C
 P 1940 5710
 F 0 "#PWR?" H 1940 5460 50  0001 C CNN
@@
 $Comp
 L power:+5V #PWR?
-U 1 1 5C4D3A94
+U 1 1 5C4E071F
 P 3040 5050
 F 0 "#PWR?" H 3040 4900 50  0001 C CNN

Commit message: Added Footprints
-Whoooo boy here we go
Parts:
- C601, C602: renamed from C?; footprint (none) -> Capacitors_SMD:C_0805_HandSoldering
- J601, J602, J603, J604: renamed from J?; footprint (none) -> EER:RingTerminal
- R601, R602: renamed from R?; footprint (none) -> Resistors_SMD:R_1206_HandSoldering
- U601: renamed from U?; footprint (none) -> EER:PSON50P140X100X40-6N
- U602: renamed from U?; footprint (none) -> EER:POWER-SO20
Changed lines of the file:
@@
 $EndDescr
 $Comp
-L EER:LN298P U?
+L EER:LN298P U602
 U 1 1 5C4E06F9
 P 5730 3140
-F 0 "U?" H 5730 4305 50  0000 C CNN
+F 0 "U602" H 5730 4305 50  0000 C CNN
 F 1 "LN298P" H 5730 4214 50  0000 C CNN
-F 2 "" H 5730 2940 50  0001 C CNN
+F 2 "EER:POWER-SO20" H 5730 2940 50  0001 C CNN
 F 3 "https://www.digikey.ca/product-detail/en/stmicroelectronics/L298P/497-1396-5-ND/585919" H 5730 2940 50  0001 C CNN
 	1    5730 3140
@@
 $EndComp
 $Comp
-L Connector:Screw_Terminal_01x01 J?
+L Connector:Screw_Terminal_01x01 J603
 U 1 1 5C4E06FB
 P 8200 2840
-F 0 "J?" H 8279 2882 50  0000 L CNN
+F 0 "J603" H 8279 2882 50  0000 L CNN
 F 1 "Screw Terminal" H 8279 2791 50  0000 L CNN
-F 2 "" H 8200 2840 50  0001 C CNN
+F 2 "EER:RingTerminal" H 8200 2840 50  0001 C CNN
 F 3 "~" H 8200 2840 50  0001 C CNN
 	1    8200 2840
@@
 	6330 2840 8000 2840
 $Comp
-L Connector:Screw_Terminal_01x01 J?
+L Connector:Screw_Terminal_01x01 J604
 U 1 1 5C4C754E
 P 8200 3040
-F 0 "J?" H 8279 3082 50  0000 L CNN
+F 0 "J604" H 8279 3082 50  0000 L CNN
 F 1 "Screw Terminal" H 8279 2991 50  0000 L CNN
-F 2 "" H 8200 3040 50  0001 C CNN
+F 2 "EER:RingTerminal" H 8200 3040 50  0001 C CNN
 F 3 "~" H 8200 3040 50  0001 C CNN
 	1    8200 3040
@@
 	6330 3040 8000 3040
 $Comp
-L Connector:Screw_Terminal_01x01 J?
+L Connector:Screw_Terminal_01x01 J602
 U 1 1 5C4C7825
 P 3260 3040
-F 0 "J?" H 3339 3082 50  0000 L CNN
+F 0 "J602" H 3339 3082 50  0000 L CNN
 F 1 "Screw Terminal" H 3339 2991 50  0000 L CNN
-F 2 "" H 3260 3040 50  0001 C CNN
+F 2 "EER:RingTerminal" H 3260 3040 50  0001 C CNN
 F 3 "~" H 3260 3040 50  0001 C CNN
 	1    3260 3040
@@
 $EndComp
 $Comp
-L Connector:Screw_Terminal_01x01 J?
+L Connector:Screw_Terminal_01x01 J601
 U 1 1 5C4C782C
 P 3260 2840
-F 0 "J?" H 3339 2882 50  0000 L CNN
+F 0 "J601" H 3339 2882 50  0000 L CNN
 F 1 "Screw Terminal" H 3339 2791 50  0000 L CNN
-F 2 "" H 3260 2840 50  0001 C CNN
+F 2 "EER:RingTerminal" H 3260 2840 50  0001 C CNN
 F 3 "~" H 3260 2840 50  0001 C CNN
 	1    3260 2840
@@
 	4500 2240 4500 2440
 $Comp
-L power:GND #PWR?
+L power:GND #PWR0154
 U 1 1 5C4E0703
 P 6980 2590
-F 0 "#PWR?" H 6980 2340 50  0001 C CNN
+F 0 "#PWR0154" H 6980 2340 50  0001 C CNN
 F 1 "GND" H 6985 2417 50  0000 C CNN
 F 2 "" H 6980 2590 50  0001 C CNN
@@
 $EndComp
 $Comp
-L power:GND #PWR?
+L power:GND #PWR0155
 U 1 1 5C4E0704
 P 4500 2600
-F 0 "#PWR?" H 4500 2350 50  0001 C CNN
+F 0 "#PWR0155" H 4500 2350 50  0001 C CNN
 F 1 "GND" H 4505 2427 50  0000 C CNN
 F 2 "" H 4500 2600 50  0001 C CNN
@@
 $EndComp
 $Comp
-L power:GND #PWR?
+L power:GND #PWR0156
 U 1 1 5C4E0707
 P 4660 4370
-F 0 "#PWR?" H 4660 4120 50  0001 C CNN
+F 0 "#PWR0156" H 4660 4120 50  0001 C CNN
 F 1 "GND" H 4665 4197 50  0000 C CNN
 F 2 "" H 4660 4370 50  0001 C CNN
@@
 $EndComp
 $Comp
-L power:GND #PWR?
+L power:GND #PWR0157
 U 1 1 5C4E0708
 P 6950 4300
-F 0 "#PWR?" H 6950 4050 50  0001 C CNN
+F 0 "#PWR0157" H 6950 4050 50  0001 C CNN
 F 1 "GND" H 6955 4127 50  0000 C CNN
 F 2 "" H 6950 4300 50  0001 C CNN
@@
 EnableB3
 $Comp
-L Device:C C?
+L Device:C C601
 U 1 1 5C4E070B
 P 3980 3490
-F 0 "C?" H 4095 3536 50  0000 L CNN
+F 0 "C601" H 4095 3536 50  0000 L CNN
 F 1 "100nF" H 4095 3445 50  0000 L CNN
-F 2 "" H 4018 3340 50  0001 C CNN
+F 2 "Capacitors_SMD:C_0805_HandSoldering" H 4018 3340 50  0001 C CNN
 F 3 "~" H 3980 3490 50  0001 C CNN
 	1    3980 3490
@@
 	3980 3240 3980 3340
 $Comp
-L power:GND #PWR?
+L power:GND #PWR0158
 U 1 1 5C4C8C0E
 P 3980 3790
-F 0 "#PWR?" H 3980 3540 50  0001 C CNN
+F 0 "#PWR0158" H 3980 3540 50  0001 C CNN
 F 1 "GND" H 3985 3617 50  0000 C CNN
 F 2 "" H 3980 3790 50  0001 C CNN
@@
 	4210 3240 3980 3240
 $Comp
-L Device:C C?
+L Device:C C602
 U 1 1 5C4E070E
 P 7320 4150
-F 0 "C?" H 7435 4196 50  0000 L CNN
+F 0 "C602" H 7435 4196 50  0000 L CNN
 F 1 "100nF" H 7435 4105 50  0000 L CNN
-F 2 "" H 7358 4000 50  0001 C CNN
+F 2 "Capacitors_SMD:C_0805_HandSoldering" H 7358 4000 50  0001 C CNN
 F 3 "~" H 7320 4150 50  0001 C CNN
 	1    7320 4150
@@
 $EndComp
 $Comp
-L power:GND #PWR?
+L power:GND #PWR0159
 U 1 1 5C4E0710
 P 7320 4450
-F 0 "#PWR?" H 7320 4200 50  0001 C CNN
+F 0 "#PWR0159" H 7320 4200 50  0001 C CNN
 F 1 "GND" H 7325 4277 50  0000 C CNN
 F 2 "" H 7320 4450 50  0001 C CNN
@@
 	7320 4300 7320 4450
 $Comp
-L power:+5V #PWR?
+L power:+5V #PWR0160
 U 1 1 5C4E0712
 P 7320 3760
-F 0 "#PWR?" H 7320 3610 50  0001 C CNN
+F 0 "#PWR0160" H 7320 3610 50  0001 C CNN
 F 1 "+5V" H 7335 3933 50  0000 C CNN
 F 2 "" H 7320 3760 50  0001 C CNN
@@
 $EndComp
 $Comp
-L power:+12V #PWR?
+L power:+12V #PWR0161
 U 1 1 5C4E0714
 P 4210 3190
-F 0 "#PWR?" H 4210 3040 50  0001 C CNN
+F 0 "#PWR0161" H 4210 3040 50  0001 C CNN
 F 1 "+12V" H 4370 3270 50  0000 C CNN
 F 2 "" H 4210 3190 50  0001 C CNN
@@
 	3460 3040 5130 3040
 $Comp
-L Device:R_US R?
+L Device:R_US R602
 U 1 1 5C4E0716
 P 6650 2440
-F 0 "R?" V 6540 2610 50  0000 C CNN
+F 0 "R602" V 6540 2610 50  0000 C CNN
 F 1 "0.5" V 6540 2280 50  0000 C CNN
-F 2 "" V 6690 2430 50  0001 C CNN
+F 2 "Resistors_SMD:R_1206_HandSoldering" V 6690 2430 50  0001 C CNN
 F 3 "~" H 6650 2440 50  0001 C CNN
 	1    6650 2440
@@
 $EndComp
 $Comp
-L Device:R_US R?
+L Device:R_US R601
 U 1 1 5C4CAD2B
 P 4810 2440
-F 0 "R?" V 4700 2610 50  0000 C CNN
+F 0 "R601" V 4700 2610 50  0000 C CNN
 F 1 "0.5" V 4700 2280 50  0000 C CNN
-F 2 "" V 4850 2430 50  0001 C CNN
+F 2 "Resistors_SMD:R_1206_HandSoldering" V 4850 2430 50  0001 C CNN
 F 3 "~" H 4810 2440 50  0001 C CNN
 	1    4810 2440
@@
 	6330 3640 6680 3640
 $Comp
-L EER:74LVC2G14 U?
+L EER:74LVC2G14 U601
 U 1 1 5C4E071B
 P 2460 5130
-F 0 "U?" H 2460 5645 50  0000 C CNN
+F 0 "U601" H 2460 5645 50  0000 C CNN
 F 1 "74LVC2G14" H 2460 5554 50  0000 C CNN
-F 2 "" H 2460 5130 50  0001 C CNN
+F 2 "EER:PSON50P140X100X40-6N" H 2460 5130 50  0001 C CNN
 F 3 "https://www.digikey.ca/product-detail/en/diodes-incorporated/74LVC2G14FZ4-7/74LVC2G14FZ4-7DICT-ND/2901046" H 2460 5130 50  0001 C CNN
 	1    2460 5130
@@
 	1940 5130 1940 5710
 $Comp
-L power:GND #PWR?
+L power:GND #PWR0162
 U 1 1 5C4E071C
 P 1940 5710
-F 0 "#PWR?" H 1940 5460 50  0001 C CNN
+F 0 "#PWR0162" H 1940 5460 50  0001 C CNN
 F 1 "GND" H 1945 5537 50  0000 C CNN
 F 2 "" H 1940 5710 50  0001 C CNN
@@
 Connection ~ 2010 5380
 $Comp
-L power:+5V #PWR?
+L power:+5V #PWR0163
 U 1 1 5C4E071F
 P 3040 5050
-F 0 "#PWR?" H 3040 4900 50  0001 C CNN
+F 0 "#PWR0163" H 3040 4900 50  0001 C CNN
 F 1 "+5V" H 3150 5120 50  0000 C CNN
 F 2 "" H 3040 5050 50  0001 C CNN
