File: PCBs/Tooling Board/Tooling Board.kicad_pcb (KiCad board)
At the start: 2 copper layers, 104.7 x 67.4 mm, 95 parts, among them J101 Screw Terminal, J102 Screw Terminal, J103 USB_B_Mini, J201 Conn_02x05_Odd_Even, J301 Conn_01x02, J302 Conn_01x02, J401 Screw Terminal, J402 Screw Terminal, J403 Screw Terminal, J404 Screw Terminal, J501 Screw Terminal, J502 Screw Terminal, J503 Screw Terminal, J504 Screw Terminal, J701 Conn_01x03, J702 Conn_01x04, J703 Conn_01x03, J801 Conn_01x02, Q301 Q1, Q302 Q_NMOS_DGS, SW201 SW_Push, U101 TLV733P, U201 ATSAMD21E18A-MFTCT-ND, U401 74LVC2G14, U402 LN298P, U501 74LVC2G14, U502 LN298P, U701 ADA_IMU, U801 CA3140AM, U802 LM2776, U803 TL081BCDG4, Y201 32.7680kHz

Commit message: Tooling Gerbs
-Respun Gerbers
Other:
- board text added: "Charity T."
- board text added: "David D."
- board text added: "Ovo"
- board text added: "Patrick W."
Changed lines of the file:
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@@
   (general
     (thickness 1.6)
-    (drawings 48)
+    (drawings 52)
     (tracks 1047)
     (zones 0)
@@
     (fp_poly (pts (xy 8.8725 1.3825) (xy 9.4325 1.3825) (xy 9.4325 1.4175) (xy 8.8725 1.4175)) (layer B.SilkS) (width 0))
   )
+  (gr_text "Patrick W." (at 115.07 64.14) (layer B.SilkS)
+    (effects (font (size 1 1) (thickness 0.25)) (justify mirror))
+  )
+  (gr_text Ovo (at 114.47 69.8) (layer B.SilkS)
+    (effects (font (size 1 1) (thickness 0.25)) (justify mirror))
+  )
+  (gr_text "Charity T." (at 114.67 67.97) (layer B.SilkS)
+    (effects (font (size 1 1) (thickness 0.25)) (justify mirror))
+  )
+  (gr_text "David D." (at 114.42 66.12) (layer B.SilkS)
+    (effects (font (size 1 1) (thickness 0.25)) (justify mirror))
+  )
   (gr_text "Mark Belbin - 2019" (at 116.82 81.13) (layer B.SilkS)
     (effects (font (size 1.5 1.5) (thickness 0.3)) (justify mirror))
@@
   (via (at 197.46 40.06) (size 6) (drill 3) (layers F.Cu B.Cu) (net 0) (status 40000))
   (via (at 107.45 40.06) (size 6) (drill 3) (layers F.Cu B.Cu) (net 0) (status 40000))
-  (via (at 169.61 57.27) (size 0.8) (drill 0.4) (layers F.Cu B.Cu) (net 2))
-  (via (at 174.22 57.9) (size 0.8) (drill 0.4) (layers F.Cu B.Cu) (net 2))
-  (via (at 170.94 56.51) (size 0.8) (drill 0.4) (layers F.Cu B.Cu) (net 2))
-  (via (at 172.81 57.02) (size 0.8) (drill 0.4) (layers F.Cu B.Cu) (net 2))
-  (via (at 171.32 58.2) (size 0.8) (drill 0.4) (layers F.Cu B.Cu) (net 2))
-  (via (at 172.73 58.96) (size 0.8) (drill 0.4) (layers F.Cu B.Cu) (net 2))
-  (via (at 170.56 59.44) (size 0.8) (drill 0.4) (layers F.Cu B.Cu) (net 2))
-  (via (at 137.17 56.32) (size 0.8) (drill 0.4) (layers F.Cu B.Cu) (net 2))
-  (via (at 138.76 58.21) (size 0.8) (drill 0.4) (layers F.Cu B.Cu) (net 2))
-  (via (at 139.22 56.56) (size 0.8) (drill 0.4) (layers F.Cu B.Cu) (net 2))
-  (via (at 141.04 57.36) (size 0.8) (drill 0.4) (layers F.Cu B.Cu) (net 2))
-  (via (at 136.95 58.24) (size 0.8) (drill 0.4) (layers F.Cu B.Cu) (net 2))
-  (via (at 140.34 59.16) (size 0.8) (drill 0.4) (layers F.Cu B.Cu) (net 2))
-  (via (at 137.68 59.71) (size 0.8) (drill 0.4) (layers F.Cu B.Cu) (net 2))
   (segment (start 130.99 78.91) (end 131.19 78.71) (width 0.25) (layer F.Cu) (net 1))
   (segment (start 130.99 78.91) (end 134.92 78.91) (width 0.2) (layer F.Cu) (net 1))
@@
   (segment (start 155.05 80.87) (end 157.755 78.165) (width 0.2) (layer F.Cu) (net 1))
   (segment (start 155.05 82.18) (end 155.05 80.87) (width 0.2) (layer F.Cu) (net 1))
+  (via (at 169.61 57.27) (size 0.8) (drill 0.4) (layers F.Cu B.Cu) (net 2))
+  (via (at 174.22 57.9) (size 0.8) (drill 0.4) (layers F.Cu B.Cu) (net 2))
+  (via (at 170.94 56.51) (size 0.8) (drill 0.4) (layers F.Cu B.Cu) (net 2))
+  (via (at 172.81 57.02) (size 0.8) (drill 0.4) (layers F.Cu B.Cu) (net 2))
+  (via (at 171.32 58.2) (size 0.8) (drill 0.4) (layers F.Cu B.Cu) (net 2))
+  (via (at 172.73 58.96) (size 0.8) (drill 0.4) (layers F.Cu B.Cu) (net 2))
+  (via (at 170.56 59.44) (size 0.8) (drill 0.4) (layers F.Cu B.Cu) (net 2))
+  (via (at 137.17 56.32) (size 0.8) (drill 0.4) (layers F.Cu B.Cu) (net 2))
+  (via (at 138.76 58.21) (size 0.8) (drill 0.4) (layers F.Cu B.Cu) (net 2))
+  (via (at 139.22 56.56) (size 0.8) (drill 0.4) (layers F.Cu B.Cu) (net 2))
+  (via (at 141.04 57.36) (size 0.8) (drill 0.4) (layers F.Cu B.Cu) (net 2))
+  (via (at 136.95 58.24) (size 0.8) (drill 0.4) (layers F.Cu B.Cu) (net 2))
+  (via (at 140.34 59.16) (size 0.8) (drill 0.4) (layers F.Cu B.Cu) (net 2))
+  (via (at 137.68 59.71) (size 0.8) (drill 0.4) (layers F.Cu B.Cu) (net 2))
   (via (at 132.55 54.21) (size 0.8) (drill 0.4) (layers F.Cu B.Cu) (net 2))
   (segment (start 132.5082 55.395) (end 132.5082 54.2518) (width 0.25) (layer F.Cu) (net 2))
