File: PCBs/Tooling Board/DCMotor1-2.sch (KiCad schematic (older format))
At the start: 10 parts

Commit message: Added Sensors
-Added pH Circuit and spec'd components
-Added Pressure sensor connecter
-Added External Temp sensor connector
-Added metal detector connector + input circuit

Need to add IMU interface now (not hard)
Parts:
- removed C?: 100nF, symbol Device:C
- removed J? (x4): Screw Terminal, symbol Connector:Screw_Terminal_01x01
- removed R?: 0.5, symbol Device:R_US
- removed U?: LN298P, symbol EER:LN298P
- added C?: 100nF, symbol Device:C
- added J? (x4): Screw Terminal, symbol Connector:Screw_Terminal_01x01
- added R?: 0.5, symbol Device:R_US
- added U?: LN298P, symbol EER:LN298P
Changed lines of the file:
@@
 $Descr A4 11693 8268
 encoding utf-8
-Sheet 4 7
+Sheet 4 8
 Title ""
 Date ""
@@
 $Comp
 L EER:LN298P U?
-U 1 1 5C4C7247
+U 1 1 5C4E06F8
 P 5730 3140
 F 0 "U?" H 5730 4305 50  0000 C CNN
@@
 $Comp
 L Connector:Screw_Terminal_01x01 J?
-U 1 1 5C4C7477
+U 1 1 5C4E06FA
 P 8200 2840
 F 0 "J?" H 8279 2882 50  0000 L CNN
@@
 $Comp
 L Connector:Screw_Terminal_01x01 J?
-U 1 1 5C4C754E
+U 1 1 5C4E06FD
 P 8200 3040
 F 0 "J?" H 8279 3082 50  0000 L CNN
@@
 $Comp
 L Connector:Screw_Terminal_01x01 J?
-U 1 1 5C4C7825
+U 1 1 5C4E06FF
 P 3260 3040
 F 0 "J?" H 3339 3082 50  0000 L CNN
@@
 $Comp
 L Connector:Screw_Terminal_01x01 J?
-U 1 1 5C4C782C
+U 1 1 5C4E0701
 P 3260 2840
 F 0 "J?" H 3339 2882 50  0000 L CNN
@@
 $Comp
 L power:GND #PWR?
-U 1 1 5C4C7C2A
+U 1 1 5C4E0706
 P 4660 4370
 F 0 "#PWR?" H 4660 4120 50  0001 C CNN
@@
 $Comp
 L Device:C C?
-U 1 1 5C4C8744
+U 1 1 5C4E070A
 P 3980 3490
 F 0 "C?" H 4095 3536 50  0000 L CNN
@@
 $Comp
 L power:GND #PWR?
-U 1 1 5C4C8C0E
+U 1 1 5C4E070D
 P 3980 3790
 F 0 "#PWR?" H 3980 3540 50  0001 C CNN
@@
 $Comp
 L power:+12V #PWR?
-U 1 1 5C4C9FF7
+U 1 1 5C4E0715
 P 4210 3190
 F 0 "#PWR?" H 4210 3040 50  0001 C CNN
@@
 $Comp
 L Device:R_US R?
-U 1 1 5C4CAD2B
+U 1 1 5C4E0719
 P 4810 2440
 F 0 "R?" V 4700 2610 50  0000 C CNN
@@
 $Comp
 L power:+5V #PWR?
-U 1 1 5C4D3A94
+U 1 1 5C4E071E
 P 3040 5050
 F 0 "#PWR?" H 3040 4900 50  0001 C CNN

Commit message: Added Footprints
-Whoooo boy here we go
Parts:
- C401, C402: renamed from C?; footprint (none) -> Capacitors_SMD:C_0805_HandSoldering
- J401, J402, J403, J404: renamed from J?; footprint (none) -> EER:RingTerminal
- R401, R402: renamed from R?; footprint (none) -> Resistors_SMD:R_1206_HandSoldering
- U401: renamed from U?; footprint (none) -> EER:PSON50P140X100X40-6N
- U402: renamed from U?; footprint (none) -> EER:POWER-SO20
Changed lines of the file:
@@
 $EndDescr
 $Comp
-L EER:LN298P U?
+L EER:LN298P U402
 U 1 1 5C4E06F8
 P 5730 3140
-F 0 "U?" H 5730 4305 50  0000 C CNN
+F 0 "U402" H 5730 4305 50  0000 C CNN
 F 1 "LN298P" H 5730 4214 50  0000 C CNN
-F 2 "" H 5730 2940 50  0001 C CNN
+F 2 "EER:POWER-SO20" H 5730 2940 50  0001 C CNN
 F 3 "https://www.digikey.ca/product-detail/en/stmicroelectronics/L298P/497-1396-5-ND/585919" H 5730 2940 50  0001 C CNN
 	1    5730 3140
@@
 $EndComp
 $Comp
-L Connector:Screw_Terminal_01x01 J?
+L Connector:Screw_Terminal_01x01 J403
 U 1 1 5C4E06FA
 P 8200 2840
-F 0 "J?" H 8279 2882 50  0000 L CNN
+F 0 "J403" H 8279 2882 50  0000 L CNN
 F 1 "Screw Terminal" H 8279 2791 50  0000 L CNN
-F 2 "" H 8200 2840 50  0001 C CNN
+F 2 "EER:RingTerminal" H 8200 2840 50  0001 C CNN
 F 3 "~" H 8200 2840 50  0001 C CNN
 	1    8200 2840
@@
 	6330 2840 8000 2840
 $Comp
-L Connector:Screw_Terminal_01x01 J?
+L Connector:Screw_Terminal_01x01 J404
 U 1 1 5C4E06FD
 P 8200 3040
-F 0 "J?" H 8279 3082 50  0000 L CNN
+F 0 "J404" H 8279 3082 50  0000 L CNN
 F 1 "Screw Terminal" H 8279 2991 50  0000 L CNN
-F 2 "" H 8200 3040 50  0001 C CNN
+F 2 "EER:RingTerminal" H 8200 3040 50  0001 C CNN
 F 3 "~" H 8200 3040 50  0001 C CNN
 	1    8200 3040
@@
 	6330 3040 8000 3040
 $Comp
-L Connector:Screw_Terminal_01x01 J?
+L Connector:Screw_Terminal_01x01 J402
 U 1 1 5C4E06FF
 P 3260 3040
-F 0 "J?" H 3339 3082 50  0000 L CNN
+F 0 "J402" H 3339 3082 50  0000 L CNN
 F 1 "Screw Terminal" H 3339 2991 50  0000 L CNN
-F 2 "" H 3260 3040 50  0001 C CNN
+F 2 "EER:RingTerminal" H 3260 3040 50  0001 C CNN
 F 3 "~" H 3260 3040 50  0001 C CNN
 	1    3260 3040
@@
 $EndComp
 $Comp
-L Connector:Screw_Terminal_01x01 J?
+L Connector:Screw_Terminal_01x01 J401
 U 1 1 5C4E0701
 P 3260 2840
-F 0 "J?" H 3339 2882 50  0000 L CNN
+F 0 "J401" H 3339 2882 50  0000 L CNN
 F 1 "Screw Terminal" H 3339 2791 50  0000 L CNN
-F 2 "" H 3260 2840 50  0001 C CNN
+F 2 "EER:RingTerminal" H 3260 2840 50  0001 C CNN
 F 3 "~" H 3260 2840 50  0001 C CNN
 	1    3260 2840
@@
 	4500 2240 4500 2440
 $Comp
-L power:GND #PWR?
+L power:GND #PWR0134
 U 1 1 5C4C7BF9
 P 6980 2590
-F 0 "#PWR?" H 6980 2340 50  0001 C CNN
+F 0 "#PWR0134" H 6980 2340 50  0001 C CNN
 F 1 "GND" H 6985 2417 50  0000 C CNN
 F 2 "" H 6980 2590 50  0001 C CNN
@@
 $EndComp
 $Comp
-L power:GND #PWR?
+L power:GND #PWR0135
 U 1 1 5C4C7C15
 P 4500 2600
-F 0 "#PWR?" H 4500 2350 50  0001 C CNN
+F 0 "#PWR0135" H 4500 2350 50  0001 C CNN
 F 1 "GND" H 4505 2427 50  0000 C CNN
 F 2 "" H 4500 2600 50  0001 C CNN
@@
 $EndComp
 $Comp
-L power:GND #PWR?
+L power:GND #PWR0136
 U 1 1 5C4E0706
 P 4660 4370
-F 0 "#PWR?" H 4660 4120 50  0001 C CNN
+F 0 "#PWR0136" H 4660 4120 50  0001 C CNN
 F 1 "GND" H 4665 4197 50  0000 C CNN
 F 2 "" H 4660 4370 50  0001 C CNN
@@
 $EndComp
 $Comp
-L power:GND #PWR?
+L power:GND #PWR0137
 U 1 1 5C4C7C7B
 P 6950 4300
-F 0 "#PWR?" H 6950 4050 50  0001 C CNN
+F 0 "#PWR0137" H 6950 4050 50  0001 C CNN
 F 1 "GND" H 6955 4127 50  0000 C CNN
 F 2 "" H 6950 4300 50  0001 C CNN
@@
 EnableB1
 $Comp
-L Device:C C?
+L Device:C C401
 U 1 1 5C4E070A
 P 3980 3490
-F 0 "C?" H 4095 3536 50  0000 L CNN
+F 0 "C401" H 4095 3536 50  0000 L CNN
 F 1 "100nF" H 4095 3445 50  0000 L CNN
-F 2 "" H 4018 3340 50  0001 C CNN
+F 2 "Capacitors_SMD:C_0805_HandSoldering" H 4018 3340 50  0001 C CNN
 F 3 "~" H 3980 3490 50  0001 C CNN
 	1    3980 3490
@@
 	3980 3240 3980 3340
 $Comp
-L power:GND #PWR?
+L power:GND #PWR0138
 U 1 1 5C4E070D
 P 3980 3790
-F 0 "#PWR?" H 3980 3540 50  0001 C CNN
+F 0 "#PWR0138" H 3980 3540 50  0001 C CNN
 F 1 "GND" H 3985 3617 50  0000 C CNN
 F 2 "" H 3980 3790 50  0001 C CNN
@@
 	4210 3240 3980 3240
 $Comp
-L Device:C C?
+L Device:C C402
 U 1 1 5C4C9D1A
 P 7320 4150
-F 0 "C?" H 7435 4196 50  0000 L CNN
+F 0 "C402" H 7435 4196 50  0000 L CNN
 F 1 "100nF" H 7435 4105 50  0000 L CNN
-F 2 "" H 7358 4000 50  0001 C CNN
+F 2 "Capacitors_SMD:C_0805_HandSoldering" H 7358 4000 50  0001 C CNN
 F 3 "~" H 7320 4150 50  0001 C CNN
 	1    7320 4150
@@
 $EndComp
 $Comp
-L power:GND #PWR?
+L power:GND #PWR0139
 U 1 1 5C4C9D20
 P 7320 4450
-F 0 "#PWR?" H 7320 4200 50  0001 C CNN
+F 0 "#PWR0139" H 7320 4200 50  0001 C CNN
 F 1 "GND" H 7325 4277 50  0000 C CNN
 F 2 "" H 7320 4450 50  0001 C CNN
@@
 	7320 4300 7320 4450
 $Comp
-L power:+5V #PWR?
+L power:+5V #PWR0140
 U 1 1 5C4C9F8F
 P 7320 3760
-F 0 "#PWR?" H 7320 3610 50  0001 C CNN
+F 0 "#PWR0140" H 7320 3610 50  0001 C CNN
 F 1 "+5V" H 7335 3933 50  0000 C CNN
 F 2 "" H 7320 3760 50  0001 C CNN
@@
 $EndComp
 $Comp
-L power:+12V #PWR?
+L power:+12V #PWR0141
 U 1 1 5C4E0715
 P 4210 3190
-F 0 "#PWR?" H 4210 3040 50  0001 C CNN
+F 0 "#PWR0141" H 4210 3040 50  0001 C CNN
 F 1 "+12V" H 4370 3270 50  0000 C CNN
 F 2 "" H 4210 3190 50  0001 C CNN
@@
 	3460 3040 5130 3040
 $Comp
-L Device:R_US R?
+L Device:R_US R402
 U 1 1 5C4CABF0
 P 6650 2440
-F 0 "R?" V 6540 2610 50  0000 C CNN
+F 0 "R402" V 6540 2610 50  0000 C CNN
 F 1 "0.5" V 6540 2280 50  0000 C CNN
-F 2 "" V 6690 2430 50  0001 C CNN
+F 2 "Resistors_SMD:R_1206_HandSoldering" V 6690 2430 50  0001 C CNN
 F 3 "~" H 6650 2440 50  0001 C CNN
 	1    6650 2440
@@
 $EndComp
 $Comp
-L Device:R_US R?
+L Device:R_US R401
 U 1 1 5C4E0719
 P 4810 2440
-F 0 "R?" V 4700 2610 50  0000 C CNN
+F 0 "R401" V 4700 2610 50  0000 C CNN
 F 1 "0.5" V 4700 2280 50  0000 C CNN
-F 2 "" V 4850 2430 50  0001 C CNN
+F 2 "Resistors_SMD:R_1206_HandSoldering" V 4850 2430 50  0001 C CNN
 F 3 "~" H 4810 2440 50  0001 C CNN
 	1    4810 2440
@@
 	6330 3640 6680 3640
 $Comp
-L EER:74LVC2G14 U?
+L EER:74LVC2G14 U401
 U 1 1 5C4CF224
 P 2460 5130
-F 0 "U?" H 2460 5645 50  0000 C CNN
+F 0 "U401" H 2460 5645 50  0000 C CNN
 F 1 "74LVC2G14" H 2460 5554 50  0000 C CNN
-F 2 "" H 2460 5130 50  0001 C CNN
+F 2 "EER:PSON50P140X100X40-6N" H 2460 5130 50  0001 C CNN
 F 3 "https://www.digikey.ca/product-detail/en/diodes-incorporated/74LVC2G14FZ4-7/74LVC2G14FZ4-7DICT-ND/2901046" H 2460 5130 50  0001 C CNN
 	1    2460 5130
@@
 	1940 5130 1940 5710
 $Comp
-L power:GND #PWR?
+L power:GND #PWR0142
 U 1 1 5C4D22A3
 P 1940 5710
-F 0 "#PWR?" H 1940 5460 50  0001 C CNN
+F 0 "#PWR0142" H 1940 5460 50  0001 C CNN
 F 1 "GND" H 1945 5537 50  0000 C CNN
 F 2 "" H 1940 5710 50  0001 C CNN
@@
 Connection ~ 2010 5380
 $Comp
-L power:+5V #PWR?
+L power:+5V #PWR0143
 U 1 1 5C4E071E
 P 3040 5050
-F 0 "#PWR?" H 3040 4900 50  0001 C CNN
+F 0 "#PWR0143" H 3040 4900 50  0001 C CNN
 F 1 "+5V" H 3150 5120 50  0000 C CNN
 F 2 "" H 3040 5050 50  0001 C CNN

Commit message: Almost Finished
-Still going, help
Parts:
- C401, C402: footprint Capacitors_SMD:C_0805_HandSoldering -> Capacitors_SMD:C_0805
- R401, R402: footprint Resistors_SMD:R_1206_HandSoldering -> Resistors_SMD:R_1206
Changed lines of the file:
@@
 F 0 "C401" H 4095 3536 50  0000 L CNN
 F 1 "100nF" H 4095 3445 50  0000 L CNN
-F 2 "Capacitors_SMD:C_0805_HandSoldering" H 4018 3340 50  0001 C CNN
+F 2 "Capacitors_SMD:C_0805" H 4018 3340 50  0001 C CNN
 F 3 "~" H 3980 3490 50  0001 C CNN
 	1    3980 3490
@@
 F 0 "C402" H 7435 4196 50  0000 L CNN
 F 1 "100nF" H 7435 4105 50  0000 L CNN
-F 2 "Capacitors_SMD:C_0805_HandSoldering" H 7358 4000 50  0001 C CNN
+F 2 "Capacitors_SMD:C_0805" H 7358 4000 50  0001 C CNN
 F 3 "~" H 7320 4150 50  0001 C CNN
 	1    7320 4150
@@
 F 0 "R402" V 6540 2610 50  0000 C CNN
 F 1 "0.5" V 6540 2280 50  0000 C CNN
-F 2 "Resistors_SMD:R_1206_HandSoldering" V 6690 2430 50  0001 C CNN
+F 2 "Resistors_SMD:R_1206" V 6690 2430 50  0001 C CNN
 F 3 "~" H 6650 2440 50  0001 C CNN
 	1    6650 2440
@@
 F 0 "R401" V 4700 2610 50  0000 C CNN
 F 1 "0.5" V 4700 2280 50  0000 C CNN
-F 2 "Resistors_SMD:R_1206_HandSoldering" V 4850 2430 50  0001 C CNN
+F 2 "Resistors_SMD:R_1206" V 4850 2430 50  0001 C CNN
 F 3 "~" H 4810 2440 50  0001 C CNN
 	1    4810 2440

Commit message: tooling board bom
Parts:
- C401, C402: Digikey (none) -> 311-1140-1-ND
- J401, J402, J403, J404: Digikey (none) -> 36-7770-ND
- R401, R402: Digikey (none) -> CSR1206FKR500CT-ND
- U401: symbol EER:74LVC2G14 -> Tooling-Board-rescue:74LVC2G14-EER
- U402: symbol EER:LN298P -> Tooling-Board-rescue:LN298P-EER
Changed lines of the file:
@@
 $EndDescr
 $Comp
-L EER:LN298P U402
+L Tooling-Board-rescue:LN298P-EER U402
 U 1 1 5C4E06F8
 P 5730 3140
@@
 F 2 "EER:RingTerminal" H 8200 2840 50  0001 C CNN
 F 3 "~" H 8200 2840 50  0001 C CNN
+F 4 "36-7770-ND" H 8200 2840 50  0001 C CNN "Digikey"
 	1    8200 2840
 	1    0    0    -1
@@
 F 2 "EER:RingTerminal" H 8200 3040 50  0001 C CNN
 F 3 "~" H 8200 3040 50  0001 C CNN
+F 4 "36-7770-ND" H 8200 3040 50  0001 C CNN "Digikey"
 	1    8200 3040
 	1    0    0    -1
@@
 F 2 "EER:RingTerminal" H 3260 3040 50  0001 C CNN
 F 3 "~" H 3260 3040 50  0001 C CNN
+F 4 "36-7770-ND" H 3260 3040 50  0001 C CNN "Digikey"
 	1    3260 3040
 	-1   0    0    1
@@
 F 2 "EER:RingTerminal" H 3260 2840 50  0001 C CNN
 F 3 "~" H 3260 2840 50  0001 C CNN
+F 4 "36-7770-ND" H 3260 2840 50  0001 C CNN "Digikey"
 	1    3260 2840
 	-1   0    0    1
@@
 F 2 "Capacitors_SMD:C_0805" H 4018 3340 50  0001 C CNN
 F 3 "~" H 3980 3490 50  0001 C CNN
+F 4 "311-1140-1-ND" H 3980 3490 50  0001 C CNN "Digikey"
 	1    3980 3490
 	1    0    0    -1
@@
 F 2 "Capacitors_SMD:C_0805" H 7358 4000 50  0001 C CNN
 F 3 "~" H 7320 4150 50  0001 C CNN
+F 4 "311-1140-1-ND" H 7320 4150 50  0001 C CNN "Digikey"
 	1    7320 4150
 	1    0    0    -1
@@
 F 2 "Resistors_SMD:R_1206" V 6690 2430 50  0001 C CNN
 F 3 "~" H 6650 2440 50  0001 C CNN
+F 4 "CSR1206FKR500CT-ND" V 6650 2440 50  0001 C CNN "Digikey"
 	1    6650 2440
 	0    1    1    0
@@
 F 2 "Resistors_SMD:R_1206" V 4850 2430 50  0001 C CNN
 F 3 "~" H 4810 2440 50  0001 C CNN
+F 4 "CSR1206FKR500CT-ND" V 4810 2440 50  0001 C CNN "Digikey"
 	1    4810 2440
 	0    1    1    0
@@
 	6330 3640 6680 3640
 $Comp
-L EER:74LVC2G14 U401
+L Tooling-Board-rescue:74LVC2G14-EER U401
 U 1 1 5C4CF224
 P 2460 5130
+AR Path="/5C4CF224" Ref="U401"  Part="1"
+AR Path="/5C4A7756/5C4C657D/5C4CF224" Ref="U401"  Part="1"
 F 0 "U401" H 2460 5645 50  0000 C CNN
 F 1 "74LVC2G14" H 2460 5554 50  0000 C CNN
