File: PCBs/Tooling Board/DCMotor3-4.sch (KiCad schematic (older format))
At the start: 10 parts

Commit message: Added Sensors
-Added pH Circuit and spec'd components
-Added Pressure sensor connecter
-Added External Temp sensor connector
-Added metal detector connector + input circuit

Need to add IMU interface now (not hard)
Parts:
- removed C?: 100nF, symbol Device:C
- removed J? (x3): Screw Terminal, symbol Connector:Screw_Terminal_01x01
- removed R? (x2): 0.5, symbol Device:R_US
- removed U?: 74LVC2G14, symbol EER:74LVC2G14
- added C?: 100nF, symbol Device:C
- added J? (x3): Screw Terminal, symbol Connector:Screw_Terminal_01x01
- added R? (x2): 0.5, symbol Device:R_US
- added U?: 74LVC2G14, symbol EER:74LVC2G14
Changed lines of the file:
@@
 $Descr A4 11693 8268
 encoding utf-8
-Sheet 5 7
+Sheet 5 8
 Title ""
 Date ""
@@
 $Comp
 L Connector:Screw_Terminal_01x01 J?
-U 1 1 5C4C754E
+U 1 1 5C4E06FC
 P 8200 3040
 F 0 "J?" H 8279 3082 50  0000 L CNN
@@
 $Comp
 L Connector:Screw_Terminal_01x01 J?
-U 1 1 5C4C7825
+U 1 1 5C4E06FE
 P 3260 3040
 F 0 "J?" H 3339 3082 50  0000 L CNN
@@
 $Comp
 L Connector:Screw_Terminal_01x01 J?
-U 1 1 5C4C782C
+U 1 1 5C4E0700
 P 3260 2840
 F 0 "J?" H 3339 2882 50  0000 L CNN
@@
 $Comp
 L power:GND #PWR?
-U 1 1 5C4C7BF9
+U 1 1 5C4E0702
 P 6980 2590
 F 0 "#PWR?" H 6980 2340 50  0001 C CNN
@@
 $Comp
 L power:GND #PWR?
-U 1 1 5C4C7C15
+U 1 1 5C4E0705
 P 4500 2600
 F 0 "#PWR?" H 4500 2350 50  0001 C CNN
@@
 $Comp
 L power:GND #PWR?
-U 1 1 5C4C7C7B
+U 1 1 5C4E0709
 P 6950 4300
 F 0 "#PWR?" H 6950 4050 50  0001 C CNN
@@
 $Comp
 L power:GND #PWR?
-U 1 1 5C4C8C0E
+U 1 1 5C4E070C
 P 3980 3790
 F 0 "#PWR?" H 3980 3540 50  0001 C CNN
@@
 $Comp
 L Device:C C?
-U 1 1 5C4C9D1A
+U 1 1 5C4E070F
 P 7320 4150
 F 0 "C?" H 7435 4196 50  0000 L CNN
@@
 $Comp
 L power:GND #PWR?
-U 1 1 5C4C9D20
+U 1 1 5C4E0711
 P 7320 4450
 F 0 "#PWR?" H 7320 4200 50  0001 C CNN
@@
 $Comp
 L power:+5V #PWR?
-U 1 1 5C4C9F8F
+U 1 1 5C4E0713
 P 7320 3760
 F 0 "#PWR?" H 7320 3610 50  0001 C CNN
@@
 $Comp
 L Device:R_US R?
-U 1 1 5C4CABF0
+U 1 1 5C4E0717
 P 6650 2440
 F 0 "R?" V 6540 2610 50  0000 C CNN
@@
 $Comp
 L Device:R_US R?
-U 1 1 5C4CAD2B
+U 1 1 5C4E0718
 P 4810 2440
 F 0 "R?" V 4700 2610 50  0000 C CNN
@@
 $Comp
 L EER:74LVC2G14 U?
-U 1 1 5C4CF224
+U 1 1 5C4E071A
 P 2460 5130
 F 0 "U?" H 2460 5645 50  0000 C CNN
@@
 $Comp
 L power:GND #PWR?
-U 1 1 5C4D22A3
+U 1 1 5C4E071D
 P 1940 5710
 F 0 "#PWR?" H 1940 5460 50  0001 C CNN

Commit message: Added Footprints
-Whoooo boy here we go
Parts:
- C501, C502: renamed from C?; footprint (none) -> Capacitors_SMD:C_0805_HandSoldering
- J501, J502, J503, J504: renamed from J?; footprint (none) -> EER:RingTerminal
- R501, R502: renamed from R?; footprint (none) -> Resistors_SMD:R_1206_HandSoldering
- U501: renamed from U?; footprint (none) -> EER:PSON50P140X100X40-6N
- U502: renamed from U?; footprint (none) -> EER:POWER-SO20
Changed lines of the file:
@@
 $EndDescr
 $Comp
-L EER:LN298P U?
+L EER:LN298P U502
 U 1 1 5C4C7247
 P 5730 3140
-F 0 "U?" H 5730 4305 50  0000 C CNN
+F 0 "U502" H 5730 4305 50  0000 C CNN
 F 1 "LN298P" H 5730 4214 50  0000 C CNN
-F 2 "" H 5730 2940 50  0001 C CNN
+F 2 "EER:POWER-SO20" H 5730 2940 50  0001 C CNN
 F 3 "https://www.digikey.ca/product-detail/en/stmicroelectronics/L298P/497-1396-5-ND/585919" H 5730 2940 50  0001 C CNN
 	1    5730 3140
@@
 $EndComp
 $Comp
-L Connector:Screw_Terminal_01x01 J?
+L Connector:Screw_Terminal_01x01 J503
 U 1 1 5C4C7477
 P 8200 2840
-F 0 "J?" H 8279 2882 50  0000 L CNN
+F 0 "J503" H 8279 2882 50  0000 L CNN
 F 1 "Screw Terminal" H 8279 2791 50  0000 L CNN
-F 2 "" H 8200 2840 50  0001 C CNN
+F 2 "EER:RingTerminal" H 8200 2840 50  0001 C CNN
 F 3 "~" H 8200 2840 50  0001 C CNN
 	1    8200 2840
@@
 	6330 2840 8000 2840
 $Comp
-L Connector:Screw_Terminal_01x01 J?
+L Connector:Screw_Terminal_01x01 J504
 U 1 1 5C4E06FC
 P 8200 3040
-F 0 "J?" H 8279 3082 50  0000 L CNN
+F 0 "J504" H 8279 3082 50  0000 L CNN
 F 1 "Screw Terminal" H 8279 2991 50  0000 L CNN
-F 2 "" H 8200 3040 50  0001 C CNN
+F 2 "EER:RingTerminal" H 8200 3040 50  0001 C CNN
 F 3 "~" H 8200 3040 50  0001 C CNN
 	1    8200 3040
@@
 	6330 3040 8000 3040
 $Comp
-L Connector:Screw_Terminal_01x01 J?
+L Connector:Screw_Terminal_01x01 J502
 U 1 1 5C4E06FE
 P 3260 3040
-F 0 "J?" H 3339 3082 50  0000 L CNN
+F 0 "J502" H 3339 3082 50  0000 L CNN
 F 1 "Screw Terminal" H 3339 2991 50  0000 L CNN
-F 2 "" H 3260 3040 50  0001 C CNN
+F 2 "EER:RingTerminal" H 3260 3040 50  0001 C CNN
 F 3 "~" H 3260 3040 50  0001 C CNN
 	1    3260 3040
@@
 $EndComp
 $Comp
-L Connector:Screw_Terminal_01x01 J?
+L Connector:Screw_Terminal_01x01 J501
 U 1 1 5C4E0700
 P 3260 2840
-F 0 "J?" H 3339 2882 50  0000 L CNN
+F 0 "J501" H 3339 2882 50  0000 L CNN
 F 1 "Screw Terminal" H 3339 2791 50  0000 L CNN
-F 2 "" H 3260 2840 50  0001 C CNN
+F 2 "EER:RingTerminal" H 3260 2840 50  0001 C CNN
 F 3 "~" H 3260 2840 50  0001 C CNN
 	1    3260 2840
@@
 	4500 2240 4500 2440
 $Comp
-L power:GND #PWR?
+L power:GND #PWR0144
 U 1 1 5C4E0702
 P 6980 2590
-F 0 "#PWR?" H 6980 2340 50  0001 C CNN
+F 0 "#PWR0144" H 6980 2340 50  0001 C CNN
 F 1 "GND" H 6985 2417 50  0000 C CNN
 F 2 "" H 6980 2590 50  0001 C CNN
@@
 $EndComp
 $Comp
-L power:GND #PWR?
+L power:GND #PWR0145
 U 1 1 5C4E0705
 P 4500 2600
-F 0 "#PWR?" H 4500 2350 50  0001 C CNN
+F 0 "#PWR0145" H 4500 2350 50  0001 C CNN
 F 1 "GND" H 4505 2427 50  0000 C CNN
 F 2 "" H 4500 2600 50  0001 C CNN
@@
 $EndComp
 $Comp
-L power:GND #PWR?
+L power:GND #PWR0146
 U 1 1 5C4C7C2A
 P 4660 4370
-F 0 "#PWR?" H 4660 4120 50  0001 C CNN
+F 0 "#PWR0146" H 4660 4120 50  0001 C CNN
 F 1 "GND" H 4665 4197 50  0000 C CNN
 F 2 "" H 4660 4370 50  0001 C CNN
@@
 $EndComp
 $Comp
-L power:GND #PWR?
+L power:GND #PWR0147
 U 1 1 5C4E0709
 P 6950 4300
-F 0 "#PWR?" H 6950 4050 50  0001 C CNN
+F 0 "#PWR0147" H 6950 4050 50  0001 C CNN
 F 1 "GND" H 6955 4127 50  0000 C CNN
 F 2 "" H 6950 4300 50  0001 C CNN
@@
 EnableB2
 $Comp
-L Device:C C?
+L Device:C C501
 U 1 1 5C4C8744
 P 3980 3490
-F 0 "C?" H 4095 3536 50  0000 L CNN
+F 0 "C501" H 4095 3536 50  0000 L CNN
 F 1 "100nF" H 4095 3445 50  0000 L CNN
-F 2 "" H 4018 3340 50  0001 C CNN
+F 2 "Capacitors_SMD:C_0805_HandSoldering" H 4018 3340 50  0001 C CNN
 F 3 "~" H 3980 3490 50  0001 C CNN
 	1    3980 3490
@@
 	3980 3240 3980 3340
 $Comp
-L power:GND #PWR?
+L power:GND #PWR0148
 U 1 1 5C4E070C
 P 3980 3790
-F 0 "#PWR?" H 3980 3540 50  0001 C CNN
+F 0 "#PWR0148" H 3980 3540 50  0001 C CNN
 F 1 "GND" H 3985 3617 50  0000 C CNN
 F 2 "" H 3980 3790 50  0001 C CNN
@@
 	4210 3240 3980 3240
 $Comp
-L Device:C C?
+L Device:C C502
 U 1 1 5C4E070F
 P 7320 4150
-F 0 "C?" H 7435 4196 50  0000 L CNN
+F 0 "C502" H 7435 4196 50  0000 L CNN
 F 1 "100nF" H 7435 4105 50  0000 L CNN
-F 2 "" H 7358 4000 50  0001 C CNN
+F 2 "Capacitors_SMD:C_0805_HandSoldering" H 7358 4000 50  0001 C CNN
 F 3 "~" H 7320 4150 50  0001 C CNN
 	1    7320 4150
@@
 $EndComp
 $Comp
-L power:GND #PWR?
+L power:GND #PWR0149
 U 1 1 5C4E0711
 P 7320 4450
-F 0 "#PWR?" H 7320 4200 50  0001 C CNN
+F 0 "#PWR0149" H 7320 4200 50  0001 C CNN
 F 1 "GND" H 7325 4277 50  0000 C CNN
 F 2 "" H 7320 4450 50  0001 C CNN
@@
 	7320 4300 7320 4450
 $Comp
-L power:+5V #PWR?
+L power:+5V #PWR0150
 U 1 1 5C4E0713
 P 7320 3760
-F 0 "#PWR?" H 7320 3610 50  0001 C CNN
+F 0 "#PWR0150" H 7320 3610 50  0001 C CNN
 F 1 "+5V" H 7335 3933 50  0000 C CNN
 F 2 "" H 7320 3760 50  0001 C CNN
@@
 $EndComp
 $Comp
-L power:+12V #PWR?
+L power:+12V #PWR0151
 U 1 1 5C4C9FF7
 P 4210 3190
-F 0 "#PWR?" H 4210 3040 50  0001 C CNN
+F 0 "#PWR0151" H 4210 3040 50  0001 C CNN
 F 1 "+12V" H 4370 3270 50  0000 C CNN
 F 2 "" H 4210 3190 50  0001 C CNN
@@
 	3460 3040 5130 3040
 $Comp
-L Device:R_US R?
+L Device:R_US R502
 U 1 1 5C4E0717
 P 6650 2440
-F 0 "R?" V 6540 2610 50  0000 C CNN
+F 0 "R502" V 6540 2610 50  0000 C CNN
 F 1 "0.5" V 6540 2280 50  0000 C CNN
-F 2 "" V 6690 2430 50  0001 C CNN
+F 2 "Resistors_SMD:R_1206_HandSoldering" V 6690 2430 50  0001 C CNN
 F 3 "~" H 6650 2440 50  0001 C CNN
 	1    6650 2440
@@
 $EndComp
 $Comp
-L Device:R_US R?
+L Device:R_US R501
 U 1 1 5C4E0718
 P 4810 2440
-F 0 "R?" V 4700 2610 50  0000 C CNN
+F 0 "R501" V 4700 2610 50  0000 C CNN
 F 1 "0.5" V 4700 2280 50  0000 C CNN
-F 2 "" V 4850 2430 50  0001 C CNN
+F 2 "Resistors_SMD:R_1206_HandSoldering" V 4850 2430 50  0001 C CNN
 F 3 "~" H 4810 2440 50  0001 C CNN
 	1    4810 2440
@@
 	6330 3640 6680 3640
 $Comp
-L EER:74LVC2G14 U?
+L EER:74LVC2G14 U501
 U 1 1 5C4E071A
 P 2460 5130
-F 0 "U?" H 2460 5645 50  0000 C CNN
+F 0 "U501" H 2460 5645 50  0000 C CNN
 F 1 "74LVC2G14" H 2460 5554 50  0000 C CNN
-F 2 "" H 2460 5130 50  0001 C CNN
+F 2 "EER:PSON50P140X100X40-6N" H 2460 5130 50  0001 C CNN
 F 3 "https://www.digikey.ca/product-detail/en/diodes-incorporated/74LVC2G14FZ4-7/74LVC2G14FZ4-7DICT-ND/2901046" H 2460 5130 50  0001 C CNN
 	1    2460 5130
@@
 	1940 5130 1940 5710
 $Comp
-L power:GND #PWR?
+L power:GND #PWR0152
 U 1 1 5C4E071D
 P 1940 5710
-F 0 "#PWR?" H 1940 5460 50  0001 C CNN
+F 0 "#PWR0152" H 1940 5460 50  0001 C CNN
 F 1 "GND" H 1945 5537 50  0000 C CNN
 F 2 "" H 1940 5710 50  0001 C CNN
@@
 Connection ~ 2010 5380
 $Comp
-L power:+5V #PWR?
+L power:+5V #PWR0153
 U 1 1 5C4D3A94
 P 3040 5050
-F 0 "#PWR?" H 3040 4900 50  0001 C CNN
+F 0 "#PWR0153" H 3040 4900 50  0001 C CNN
 F 1 "+5V" H 3150 5120 50  0000 C CNN
 F 2 "" H 3040 5050 50  0001 C CNN

Commit message: Almost Finished
-Still going, help
Parts:
- C501, C502: footprint Capacitors_SMD:C_0805_HandSoldering -> Capacitors_SMD:C_0805
- R501, R502: footprint Resistors_SMD:R_1206_HandSoldering -> Resistors_SMD:R_1206
Changed lines of the file:
@@
 F 0 "C501" H 4095 3536 50  0000 L CNN
 F 1 "100nF" H 4095 3445 50  0000 L CNN
-F 2 "Capacitors_SMD:C_0805_HandSoldering" H 4018 3340 50  0001 C CNN
+F 2 "Capacitors_SMD:C_0805" H 4018 3340 50  0001 C CNN
 F 3 "~" H 3980 3490 50  0001 C CNN
 	1    3980 3490
@@
 F 0 "C502" H 7435 4196 50  0000 L CNN
 F 1 "100nF" H 7435 4105 50  0000 L CNN
-F 2 "Capacitors_SMD:C_0805_HandSoldering" H 7358 4000 50  0001 C CNN
+F 2 "Capacitors_SMD:C_0805" H 7358 4000 50  0001 C CNN
 F 3 "~" H 7320 4150 50  0001 C CNN
 	1    7320 4150
@@
 F 0 "R502" V 6540 2610 50  0000 C CNN
 F 1 "0.5" V 6540 2280 50  0000 C CNN
-F 2 "Resistors_SMD:R_1206_HandSoldering" V 6690 2430 50  0001 C CNN
+F 2 "Resistors_SMD:R_1206" V 6690 2430 50  0001 C CNN
 F 3 "~" H 6650 2440 50  0001 C CNN
 	1    6650 2440
@@
 F 0 "R501" V 4700 2610 50  0000 C CNN
 F 1 "0.5" V 4700 2280 50  0000 C CNN
-F 2 "Resistors_SMD:R_1206_HandSoldering" V 4850 2430 50  0001 C CNN
+F 2 "Resistors_SMD:R_1206" V 4850 2430 50  0001 C CNN
 F 3 "~" H 4810 2440 50  0001 C CNN
 	1    4810 2440

Commit message: tooling board bom
Parts:
- C501, C502: Digikey (none) -> 311-1140-1-ND
- J501, J502, J503, J504: Digikey (none) -> 36-7770-ND
- R501, R502: Digikey (none) -> CSR1206FKR500CT-ND
- U501: symbol EER:74LVC2G14 -> Tooling-Board-rescue:74LVC2G14-EER
- U502: symbol EER:LN298P -> Tooling-Board-rescue:LN298P-EER
Changed lines of the file:
@@
 $EndDescr
 $Comp
-L EER:LN298P U502
+L Tooling-Board-rescue:LN298P-EER U502
 U 1 1 5C4C7247
 P 5730 3140
@@
 F 2 "EER:RingTerminal" H 8200 2840 50  0001 C CNN
 F 3 "~" H 8200 2840 50  0001 C CNN
+F 4 "36-7770-ND" H 8200 2840 50  0001 C CNN "Digikey"
 	1    8200 2840
 	1    0    0    -1
@@
 F 2 "EER:RingTerminal" H 8200 3040 50  0001 C CNN
 F 3 "~" H 8200 3040 50  0001 C CNN
+F 4 "36-7770-ND" H 8200 3040 50  0001 C CNN "Digikey"
 	1    8200 3040
 	1    0    0    -1
@@
 F 2 "EER:RingTerminal" H 3260 3040 50  0001 C CNN
 F 3 "~" H 3260 3040 50  0001 C CNN
+F 4 "36-7770-ND" H 3260 3040 50  0001 C CNN "Digikey"
 	1    3260 3040
 	-1   0    0    1
@@
 F 2 "EER:RingTerminal" H 3260 2840 50  0001 C CNN
 F 3 "~" H 3260 2840 50  0001 C CNN
+F 4 "36-7770-ND" H 3260 2840 50  0001 C CNN "Digikey"
 	1    3260 2840
 	-1   0    0    1
@@
 F 2 "Capacitors_SMD:C_0805" H 4018 3340 50  0001 C CNN
 F 3 "~" H 3980 3490 50  0001 C CNN
+F 4 "311-1140-1-ND" H 3980 3490 50  0001 C CNN "Digikey"
 	1    3980 3490
 	1    0    0    -1
@@
 F 2 "Capacitors_SMD:C_0805" H 7358 4000 50  0001 C CNN
 F 3 "~" H 7320 4150 50  0001 C CNN
+F 4 "311-1140-1-ND" H 7320 4150 50  0001 C CNN "Digikey"
 	1    7320 4150
 	1    0    0    -1
@@
 F 2 "Resistors_SMD:R_1206" V 6690 2430 50  0001 C CNN
 F 3 "~" H 6650 2440 50  0001 C CNN
+F 4 "CSR1206FKR500CT-ND" V 6650 2440 50  0001 C CNN "Digikey"
 	1    6650 2440
 	0    1    1    0
@@
 F 2 "Resistors_SMD:R_1206" V 4850 2430 50  0001 C CNN
 F 3 "~" H 4810 2440 50  0001 C CNN
+F 4 "CSR1206FKR500CT-ND" V 4810 2440 50  0001 C CNN "Digikey"
 	1    4810 2440
 	0    1    1    0
@@
 	6330 3640 6680 3640
 $Comp
-L EER:74LVC2G14 U501
+L Tooling-Board-rescue:74LVC2G14-EER U501
 U 1 1 5C4E071A
 P 2460 5130
+AR Path="/5C4E071A" Ref="U501"  Part="1"
+AR Path="/5C4A7756/5C4D499E/5C4E071A" Ref="U501"  Part="1"
 F 0 "U501" H 2460 5645 50  0000 C CNN
 F 1 "74LVC2G14" H 2460 5554 50  0000 C CNN
