File: PCBs/Tooling Board/Sensors.sch (KiCad schematic (older format))
At the start: 0 parts

Commit message: Added Sensors
-Added pH Circuit and spec'd components
-Added Pressure sensor connecter
-Added External Temp sensor connector
-Added metal detector connector + input circuit

Need to add IMU interface now (not hard)
Parts:
- added C?: 1uF, symbol Device:C
- added J?: Conn_01x04, symbol Connector_Generic:Conn_01x04
- added J? (x2): Conn_01x03, symbol Connector_Generic:Conn_01x03
- added R?: 4.7k, symbol Device:R_US
- added R?: 75k, symbol Device:R_US
- added R?: 25k, symbol Device:R_US
Connections:
- new net: C?.1, J?.2 (Pin_2), R?.2
- new net +12V: J?.1 (Pin_1)
- new net +3V3: J?.1 (Pin_1), R?.1
- new net +5V: J?.1 (Pin_1)
- new net GND: C?.2, J?.3 (Pin_3), J?.3 (Pin_3), J?.4 (Pin_4), R?.1
- new net SCL: J?.3 (Pin_3)
- new net SDA: J?.2 (Pin_2)
- new net T_DATA: J?.2 (Pin_2), R?.2
- new net V_METAL: R?.1, R?.2
Other:
- note added: "Extra Pins"
- note added: "IMU"
- note added: "Metal Detector"
- note added: "Pressure Sensor"
- note added: "Sensors"
- note added: "Temperature Sensor"
- note added: "pH Sensor"

Commit message: Added IMU
-Added schematic and configuration for IMU.
-Still need to create a footprint
Parts:
- added U?: ADA_IMU, symbol EER:ADA_IMU
Connections:
- wire segments 28 -> 36
- no-connect marks 0 -> 5
Changed lines of the file:
@@
 	1    0    0    -1
 $EndComp
+$Comp
+L EER:ADA_IMU U?
+U 1 1 5C56FA6A
+P 5060 2000
+F 0 "U?" H 5060 2665 50  0000 C CNN
+F 1 "ADA_IMU" H 5060 2574 50  0000 C CNN
+F 2 "" H 5060 2000 50  0001 C CNN
+F 3 "" H 5060 2000 50  0001 C CNN
+	1    5060 2000
+	1    0    0    -1
+$EndComp
+Wire Wire Line
+	4660 1600 4550 1600
+Wire Wire Line
+	4550 1600 4550 1500
+$Comp
+L power:+3V3 #PWR?
+U 1 1 5C56FF97
+P 4550 1500
+F 0 "#PWR?" H 4550 1350 50  0001 C CNN
+F 1 "+3V3" H 4565 1673 50  0000 C CNN
+F 2 "" H 4550 1500 50  0001 C CNN
+F 3 "" H 4550 1500 50  0001 C CNN
+	1    4550 1500
+	1    0    0    -1
+$EndComp
+NoConn ~ 5460 1750
+NoConn ~ 5460 1900
+NoConn ~ 5460 2100
+NoConn ~ 5460 2250
+Wire Wire Line
+	4660 2100 4400 2100
+Wire Wire Line
+	4660 2250 4400 2250
+Text GLabel 4400 2100 0    50   Input ~ 0
+SDA
+Text GLabel 4400 2250 0    50   Input ~ 0
+SCL
+Wire Wire Line
+	4660 2400 4590 2400
+$Comp
+L power:GND #PWR?
+U 1 1 5C5728C0
+P 4590 2610
+F 0 "#PWR?" H 4590 2360 50  0001 C CNN
+F 1 "GND" H 4595 2437 50  0000 C CNN
+F 2 "" H 4590 2610 50  0001 C CNN
+F 3 "" H 4590 2610 50  0001 C CNN
+	1    4590 2610
+	1    0    0    -1
+$EndComp
+Wire Wire Line
+	4660 1900 4590 1900
+Wire Wire Line
+	4590 1900 4590 2400
+Connection ~ 4590 2400
+Wire Wire Line
+	4590 2400 4590 2610
+NoConn ~ 4660 1750
 $EndSCHEMATC

Commit message: Added Footprints
-Whoooo boy here we go
Parts:
- C701: renamed from C?; footprint (none) -> Capacitors_SMD:C_0805_HandSoldering
- J701, J703: renamed from J?; footprint (none) -> Junction Box:70553-03
- J702: renamed from J?; footprint (none) -> Junction Box:70553-04
- R701, R702, R703: renamed from R?; footprint (none) -> Resistors_SMD:R_0805_HandSoldering
- U701: renamed from U?; footprint (none) -> EER:IMU
Changed lines of the file:
@@
 Extra Pins
 $Comp
-L Connector_Generic:Conn_01x04 J?
+L Connector_Generic:Conn_01x04 J702
 U 1 1 5C4E1094
 P 9750 4910
-F 0 "J?" H 9830 4902 50  0000 L CNN
+F 0 "J702" H 9830 4902 50  0000 L CNN
 F 1 "Conn_01x04" H 9830 4811 50  0000 L CNN
-F 2 "" H 9750 4910 50  0001 C CNN
+F 2 "Junction Box:70553-04" H 9750 4910 50  0001 C CNN
 F 3 "~" H 9750 4910 50  0001 C CNN
 	1    9750 4910
@@
 	9420 5110 9420 5250
 $Comp
-L power:+5V #PWR?
+L power:+5V #PWR0164
 U 1 1 5C4E12E2
 P 9410 4700
-F 0 "#PWR?" H 9410 4550 50  0001 C CNN
+F 0 "#PWR0164" H 9410 4550 50  0001 C CNN
 F 1 "+5V" H 9425 4873 50  0000 C CNN
 F 2 "" H 9410 4700 50  0001 C CNN
@@
 $EndComp
 $Comp
-L power:GND #PWR?
+L power:GND #PWR0165
 U 1 1 5C4E130D
 P 9420 5250
-F 0 "#PWR?" H 9420 5000 50  0001 C CNN
+F 0 "#PWR0165" H 9420 5000 50  0001 C CNN
 F 1 "GND" H 9425 5077 50  0000 C CNN
 F 2 "" H 9420 5250 50  0001 C CNN
@@
 SCL
 $Comp
-L Connector_Generic:Conn_01x03 J?
+L Connector_Generic:Conn_01x03 J701
 U 1 1 5C4FD052
 P 9730 3420
-F 0 "J?" H 9810 3462 50  0000 L CNN
+F 0 "J701" H 9810 3462 50  0000 L CNN
 F 1 "Conn_01x03" H 9810 3371 50  0000 L CNN
-F 2 "" H 9730 3420 50  0001 C CNN
+F 2 "Junction Box:70553-03" H 9730 3420 50  0001 C CNN
 F 3 "~" H 9730 3420 50  0001 C CNN
 	1    9730 3420
@@
 	9410 3520 9410 3700
 $Comp
-L power:GND #PWR?
+L power:GND #PWR0166
 U 1 1 5C4FD201
 P 9410 3700
-F 0 "#PWR?" H 9410 3450 50  0001 C CNN
+F 0 "#PWR0166" H 9410 3450 50  0001 C CNN
 F 1 "GND" H 9415 3527 50  0000 C CNN
 F 2 "" H 9410 3700 50  0001 C CNN
@@
 T_DATA
 $Comp
-L power:+3V3 #PWR?
+L power:+3V3 #PWR0167
 U 1 1 5C4FD472
 P 9410 3190
-F 0 "#PWR?" H 9410 3040 50  0001 C CNN
+F 0 "#PWR0167" H 9410 3040 50  0001 C CNN
 F 1 "+3V3" H 9425 3363 50  0000 C CNN
 F 2 "" H 9410 3190 50  0001 C CNN
@@
 $EndComp
 $Comp
-L Device:R_US R?
+L Device:R_US R703
 U 1 1 5C4FD49F
 P 9210 3320
-F 0 "R?" V 9005 3320 50  0000 C CNN
+F 0 "R703" V 9005 3320 50  0000 C CNN
 F 1 "4.7k" V 9096 3320 50  0000 C CNN
-F 2 "" V 9250 3310 50  0001 C CNN
+F 2 "Resistors_SMD:R_0805_HandSoldering" V 9250 3310 50  0001 C CNN
 F 3 "~" H 9210 3320 50  0001 C CNN
 	1    9210 3320
@@
 Connection ~ 9410 3320
 $Comp
-L Connector_Generic:Conn_01x03 J?
+L Connector_Generic:Conn_01x03 J703
 U 1 1 5C4FDAEC
 P 9780 1690
-F 0 "J?" H 9860 1732 50  0000 L CNN
+F 0 "J703" H 9860 1732 50  0000 L CNN
 F 1 "Conn_01x03" H 9860 1641 50  0000 L CNN
-F 2 "" H 9780 1690 50  0001 C CNN
+F 2 "Junction Box:70553-03" H 9780 1690 50  0001 C CNN
 F 3 "~" H 9780 1690 50  0001 C CNN
 	1    9780 1690
@@
 	8700 1690 8700 1780
 $Comp
-L Device:R_US R?
+L Device:R_US R701
 U 1 1 5C4FE095
 P 8700 1930
-F 0 "R?" H 8632 1884 50  0000 R CNN
+F 0 "R701" H 8632 1884 50  0000 R CNN
 F 1 "75k" H 8632 1975 50  0000 R CNN
-F 2 "" V 8740 1920 50  0001 C CNN
+F 2 "Resistors_SMD:R_0805_HandSoldering" V 8740 1920 50  0001 C CNN
 F 3 "~" H 8700 1930 50  0001 C CNN
 	1    8700 1930
@@
 $EndComp
 $Comp
-L Device:R_US R?
+L Device:R_US R702
 U 1 1 5C4FE116
 P 8700 2260
-F 0 "R?" H 8632 2214 50  0000 R CNN
+F 0 "R702" H 8632 2214 50  0000 R CNN
 F 1 "25k" H 8632 2305 50  0000 R CNN
-F 2 "" V 8740 2250 50  0001 C CNN
+F 2 "Resistors_SMD:R_0805_HandSoldering" V 8740 2250 50  0001 C CNN
 F 3 "~" H 8700 2260 50  0001 C CNN
 	1    8700 2260
@@
 $EndComp
 $Comp
-L power:+12V #PWR?
+L power:+12V #PWR0168
 U 1 1 5C4FE600
 P 9410 1410
-F 0 "#PWR?" H 9410 1260 50  0001 C CNN
+F 0 "#PWR0168" H 9410 1260 50  0001 C CNN
 F 1 "+12V" H 9425 1583 50  0000 C CNN
 F 2 "" H 9410 1410 50  0001 C CNN
@@
 $EndComp
 $Comp
-L power:GND #PWR?
+L power:GND #PWR0169
 U 1 1 5C4FE61E
 P 9410 1950
-F 0 "#PWR?" H 9410 1700 50  0001 C CNN
+F 0 "#PWR0169" H 9410 1700 50  0001 C CNN
 F 1 "GND" H 9415 1777 50  0000 C CNN
 F 2 "" H 9410 1950 50  0001 C CNN
@@
 $EndComp
 $Comp
-L power:GND #PWR?
+L power:GND #PWR0170
 U 1 1 5C4FE677
 P 8700 2460
-F 0 "#PWR?" H 8700 2210 50  0001 C CNN
+F 0 "#PWR0170" H 8700 2210 50  0001 C CNN
 F 1 "GND" H 8705 2287 50  0000 C CNN
 F 2 "" H 8700 2460 50  0001 C CNN
@@
 V_METAL
 $Comp
-L Device:C C?
+L Device:C C701
 U 1 1 5C4FF49D
 P 9070 1920
-F 0 "C?" H 9185 1966 50  0000 L CNN
+F 0 "C701" H 9185 1966 50  0000 L CNN
 F 1 "1uF" H 9185 1875 50  0000 L CNN
-F 2 "" H 9108 1770 50  0001 C CNN
+F 2 "Capacitors_SMD:C_0805_HandSoldering" H 9108 1770 50  0001 C CNN
 F 3 "~" H 9070 1920 50  0001 C CNN
 	1    9070 1920
@@
 	9070 2070 9070 2200
 $Comp
-L power:GND #PWR?
+L power:GND #PWR0171
 U 1 1 5C500307
 P 9070 2200
-F 0 "#PWR?" H 9070 1950 50  0001 C CNN
+F 0 "#PWR0171" H 9070 1950 50  0001 C CNN
 F 1 "GND" H 9075 2027 50  0000 C CNN
 F 2 "" H 9070 2200 50  0001 C CNN
@@
 $EndComp
 $Comp
-L EER:ADA_IMU U?
+L EER:ADA_IMU U701
 U 1 1 5C56FA6A
 P 5060 2000
-F 0 "U?" H 5060 2665 50  0000 C CNN
+F 0 "U701" H 5060 2665 50  0000 C CNN
 F 1 "ADA_IMU" H 5060 2574 50  0000 C CNN
-F 2 "" H 5060 2000 50  0001 C CNN
+F 2 "EER:IMU" H 5060 2000 50  0001 C CNN
 F 3 "" H 5060 2000 50  0001 C CNN
 	1    5060 2000
@@
 	4550 1600 4550 1500
 $Comp
-L power:+3V3 #PWR?
+L power:+3V3 #PWR0172
 U 1 1 5C56FF97
 P 4550 1500
-F 0 "#PWR?" H 4550 1350 50  0001 C CNN
+F 0 "#PWR0172" H 4550 1350 50  0001 C CNN
 F 1 "+3V3" H 4565 1673 50  0000 C CNN
 F 2 "" H 4550 1500 50  0001 C CNN
@@
 	4660 2400 4590 2400
 $Comp
-L power:GND #PWR?
+L power:GND #PWR0173
 U 1 1 5C5728C0
 P 4590 2610
-F 0 "#PWR?" H 4590 2360 50  0001 C CNN
+F 0 "#PWR0173" H 4590 2360 50  0001 C CNN
 F 1 "GND" H 4595 2437 50  0000 C CNN
 F 2 "" H 4590 2610 50  0001 C CNN

Commit message: Almost Finished
-Still going, help
Parts:
- C701: footprint Capacitors_SMD:C_0805_HandSoldering -> Capacitors_SMD:C_0805
- J701, J703: footprint Junction Box:70553-03 -> EER:1x3_molex_llc
- J702: footprint Junction Box:70553-04 -> EER:1x4_molex_llc
- R701, R702, R703: footprint Resistors_SMD:R_0805_HandSoldering -> Resistors_SMD:R_0805
Connections:
- wire segments 36 -> 38
- no-connect marks 5 -> 4
Changed lines of the file:
@@
 $Descr A4 11693 8268
 encoding utf-8
-Sheet 7 7
+Sheet 6 7
 Title ""
 Date ""
@@
 F 0 "J702" H 9830 4902 50  0000 L CNN
 F 1 "Conn_01x04" H 9830 4811 50  0000 L CNN
-F 2 "Junction Box:70553-04" H 9750 4910 50  0001 C CNN
+F 2 "EER:1x4_molex_llc" H 9750 4910 50  0001 C CNN
 F 3 "~" H 9750 4910 50  0001 C CNN
 	1    9750 4910
@@
 F 0 "J701" H 9810 3462 50  0000 L CNN
 F 1 "Conn_01x03" H 9810 3371 50  0000 L CNN
-F 2 "Junction Box:70553-03" H 9730 3420 50  0001 C CNN
+F 2 "EER:1x3_molex_llc" H 9730 3420 50  0001 C CNN
 F 3 "~" H 9730 3420 50  0001 C CNN
 	1    9730 3420
@@
 F 0 "R703" V 9005 3320 50  0000 C CNN
 F 1 "4.7k" V 9096 3320 50  0000 C CNN
-F 2 "Resistors_SMD:R_0805_HandSoldering" V 9250 3310 50  0001 C CNN
+F 2 "Resistors_SMD:R_0805" V 9250 3310 50  0001 C CNN
 F 3 "~" H 9210 3320 50  0001 C CNN
 	1    9210 3320
@@
 F 0 "J703" H 9860 1732 50  0000 L CNN
 F 1 "Conn_01x03" H 9860 1641 50  0000 L CNN
-F 2 "Junction Box:70553-03" H 9780 1690 50  0001 C CNN
+F 2 "EER:1x3_molex_llc" H 9780 1690 50  0001 C CNN
 F 3 "~" H 9780 1690 50  0001 C CNN
 	1    9780 1690
@@
 F 0 "R701" H 8632 1884 50  0000 R CNN
 F 1 "75k" H 8632 1975 50  0000 R CNN
-F 2 "Resistors_SMD:R_0805_HandSoldering" V 8740 1920 50  0001 C CNN
+F 2 "Resistors_SMD:R_0805" V 8740 1920 50  0001 C CNN
 F 3 "~" H 8700 1930 50  0001 C CNN
 	1    8700 1930
@@
 F 0 "R702" H 8632 2214 50  0000 R CNN
 F 1 "25k" H 8632 2305 50  0000 R CNN
-F 2 "Resistors_SMD:R_0805_HandSoldering" V 8740 2250 50  0001 C CNN
+F 2 "Resistors_SMD:R_0805" V 8740 2250 50  0001 C CNN
 F 3 "~" H 8700 2260 50  0001 C CNN
 	1    8700 2260
@@
 F 0 "C701" H 9185 1966 50  0000 L CNN
 F 1 "1uF" H 9185 1875 50  0000 L CNN
-F 2 "Capacitors_SMD:C_0805_HandSoldering" H 9108 1770 50  0001 C CNN
+F 2 "Capacitors_SMD:C_0805" H 9108 1770 50  0001 C CNN
 F 3 "~" H 9070 1920 50  0001 C CNN
 	1    9070 1920
@@
 NoConn ~ 5460 1900
 NoConn ~ 5460 2100
-NoConn ~ 5460 2250
 Wire Wire Line
 	4660 2100 4400 2100
@@
 	4590 2400 4590 2610
 NoConn ~ 4660 1750
+Wire Wire Line
+	5460 2250 5650 2250
+Wire Wire Line
+	5650 2250 5650 2170
+$Comp
+L power:+3V3 #PWR?
+U 1 1 5C4E87C6
+P 5650 2170
+F 0 "#PWR?" H 5650 2020 50  0001 C CNN
+F 1 "+3V3" H 5665 2343 50  0000 C CNN
+F 2 "" H 5650 2170 50  0001 C CNN
+F 3 "" H 5650 2170 50  0001 C CNN
+	1    5650 2170
+	1    0    0    -1
+$EndComp
 $EndSCHEMATC

Commit message: tooling board bom
Parts:
- J701, J703: Digikey (none) -> WM4801-ND
- J702: Digikey (none) -> WM4802-ND
- R701: Digikey (none) -> YAG3750CT-ND
- R702: Digikey (none) -> A121556CT-ND
- R703: Digikey (none) -> 311-4.70KCRCT-ND
- U701: symbol EER:ADA_IMU -> Tooling-Board-rescue:ADA_IMU-EER
Changed lines of the file:
@@
 F 2 "EER:1x4_molex_llc" H 9750 4910 50  0001 C CNN
 F 3 "~" H 9750 4910 50  0001 C CNN
+F 4 "WM4802-ND" H 9750 4910 50  0001 C CNN "Digikey"
 	1    9750 4910
 	1    0    0    -1
@@
 F 2 "EER:1x3_molex_llc" H 9730 3420 50  0001 C CNN
 F 3 "~" H 9730 3420 50  0001 C CNN
+F 4 "WM4801-ND" H 9730 3420 50  0001 C CNN "Digikey"
 	1    9730 3420
 	1    0    0    -1
@@
 F 2 "Resistors_SMD:R_0805" V 9250 3310 50  0001 C CNN
 F 3 "~" H 9210 3320 50  0001 C CNN
+F 4 "311-4.70KCRCT-ND" V 9210 3320 50  0001 C CNN "Digikey"
 	1    9210 3320
 	0    1    1    0
@@
 F 2 "EER:1x3_molex_llc" H 9780 1690 50  0001 C CNN
 F 3 "~" H 9780 1690 50  0001 C CNN
+F 4 "WM4801-ND" H 9780 1690 50  0001 C CNN "Digikey"
 	1    9780 1690
 	1    0    0    -1
@@
 F 2 "Resistors_SMD:R_0805" V 8740 1920 50  0001 C CNN
 F 3 "~" H 8700 1930 50  0001 C CNN
+F 4 "YAG3750CT-ND" H 8700 1930 50  0001 C CNN "Digikey"
 	1    8700 1930
 	-1   0    0    1
@@
 F 2 "Resistors_SMD:R_0805" V 8740 2250 50  0001 C CNN
 F 3 "~" H 8700 2260 50  0001 C CNN
+F 4 "A121556CT-ND" H 8700 2260 50  0001 C CNN "Digikey"
 	1    8700 2260
 	-1   0    0    1
@@
 $EndComp
 $Comp
-L EER:ADA_IMU U701
+L Tooling-Board-rescue:ADA_IMU-EER U701
 U 1 1 5C56FA6A
 P 5060 2000
