File: PCBs/Tooling Board/Tooling Board.sch (KiCad schematic (older format))
At the start: 14 parts, among them J101 Screw Terminal, J102 Screw Terminal, J103 USB_B_Mini, U101 TLV733P

Commit message: tooling board bom
Parts:
- C101, C102, C104: Digikey (none) -> 399-13664-ND
- C103, C106: Digikey (none) -> 1276-6470-1-ND
- C105: Digikey (none) -> 1276-2872-1-ND
- C107: Digikey (none) -> 311-1140-1-ND
- D101: Digikey (none) -> 732-4982-1-ND
- F101: Digikey (none) -> 507-1075-1-ND
- J101, J102: Digikey (none) -> 36-7770-ND
- J103: Digikey (none) -> 151-1206-1-ND
- R101: Digikey (none) -> YAG1820CT-ND
- U101: Digikey (none) -> 296-40673-1-ND
Changed lines of the file:
@@
 F 2 "EER:RingTerminal" H 1300 1550 50  0001 C CNN
 F 3 "~" H 1300 1550 50  0001 C CNN
+F 4 "36-7770-ND" H 1300 1550 50  0001 C CNN "Digikey"
 	1    1300 1550
 	-1   0    0    1
@@
 F 2 "EER:RingTerminal" H 1300 1900 50  0001 C CNN
 F 3 "~" H 1300 1900 50  0001 C CNN
+F 4 "36-7770-ND" H 1300 1900 50  0001 C CNN "Digikey"
 	1    1300 1900
 	-1   0    0    1
@@
 F 2 "EER:32005-201" H 1670 3090 50  0001 C CNN
 F 3 "~" H 1670 3090 50  0001 C CNN
+F 4 "151-1206-1-ND" H 1520 3140 50  0001 C CNN "Digikey"
 	1    1520 3140
 	1    0    0    -1
@@
 F 1 "500mA" V 2124 2940 50  0000 C CNN
 F 2 "EER:Fuse_SMD1206_Reflow" V 2160 2940 50  0001 C CNN
-F 3 "~" H 2230 2940 50  0001 C CNN
+F 3 "https://belfuse.com/resources/datasheets/circuitprotection/ds-cp-c1q-series.pdf" H 2230 2940 50  0001 C CNN
+F 4 "507-1075-1-ND" V 2230 2940 50  0001 C CNN "Digikey"
 	1    2230 2940
 	0    1    1    0
@@
 F 1 "TLV733P" H 3000 3291 50  0000 C CNN
 F 2 "TO_SOT_Packages_SMD:SOT-23-5" H 3000 3365 50  0001 C CIN
-F 3 "296-40673-1-ND" H 3000 3090 50  0001 C CNN
+F 3 "" H 3000 3090 50  0001 C CNN
+F 4 "296-40673-1-ND" H 3000 3040 50  0001 C CNN "Digikey"
 	1    3000 3040
 	1    0    0    -1
@@
 F 1 "1uF" H 2615 3195 50  0000 L CNN
 F 2 "Capacitors_SMD:C_0805" H 2538 3090 50  0001 C CNN
-F 3 "~" H 2500 3240 50  0001 C CNN
+F 3 "http://www.samsungsem.com/kr/support/product-search/mlcc/__icsFiles/afieldfile/2018/07/23/CL21B105KBFNNNG.pdf" H 2500 3240 50  0001 C CNN
+F 4 "1276-6470-1-ND" H 2500 3240 50  0001 C CNN "Digikey"
 	1    2500 3240
 	1    0    0    -1
@@
 F 1 "10uF" H 3525 3185 50  0000 L CNN
 F 2 "Capacitors_SMD:C_0805" H 3448 3080 50  0001 C CNN
-F 3 "~" H 3410 3230 50  0001 C CNN
+F 3 "http://www.samsungsem.com/kr/support/product-search/mlcc/__icsFiles/afieldfile/2018/07/23/CL21B106KOQNNNE.pdf" H 3410 3230 50  0001 C CNN
+F 4 "1276-2872-1-ND" H 3410 3230 50  0001 C CNN "Digikey"
 	1    3410 3230
 	1    0    0    -1
@@
 F 1 "1uF" H 3955 3185 50  0000 L CNN
 F 2 "Capacitors_SMD:C_0805" H 3878 3080 50  0001 C CNN
-F 3 "~" H 3840 3230 50  0001 C CNN
+F 3 "http://www.samsungsem.com/kr/support/product-search/mlcc/__icsFiles/afieldfile/2018/07/23/CL21B105KBFNNNG.pdf" H 3840 3230 50  0001 C CNN
+F 4 "1276-6470-1-ND" H 3840 3230 50  0001 C CNN "Digikey"
 	1    3840 3230
 	1    0    0    -1
@@
 F 1 "0.1uF" H 4335 3185 50  0000 L CNN
 F 2 "Capacitors_SMD:C_0805" H 4258 3080 50  0001 C CNN
-F 3 "~" H 4220 3230 50  0001 C CNN
+F 3 "http://www.yageo.com/documents/recent/UPY-GPHC_X7R_6.3V-to-50V_18.pdf" H 4220 3230 50  0001 C CNN
+F 4 "311-1140-1-ND" H 4220 3230 50  0001 C CNN "Digikey"
 	1    4220 3230
 	1    0    0    -1
@@
 F 1 "220uF" H 2065 1675 50  0000 L CNN
 F 2 "Capacitors_THT:CP_Radial_D6.3mm_P2.50mm" H 1988 1570 50  0001 C CNN
-F 3 "~" H 1950 1720 50  0001 C CNN
+F 3 "https://content.kemet.com/datasheets/KEM_A4067_A750.pdf" H 1950 1720 50  0001 C CNN
+F 4 "399-13664-ND" H 1950 1720 50  0001 C CNN "Digikey"
 	1    1950 1720
 	1    0    0    -1
@@
 F 1 "220uF" H 2525 1675 50  0000 L CNN
 F 2 "Capacitors_THT:CP_Radial_D6.3mm_P2.50mm" H 2448 1570 50  0001 C CNN
-F 3 "~" H 2410 1720 50  0001 C CNN
+F 3 "https://content.kemet.com/datasheets/KEM_A4067_A750.pdf" H 2410 1720 50  0001 C CNN
+F 4 "399-13664-ND" H 2410 1720 50  0001 C CNN "Digikey"
 	1    2410 1720
 	1    0    0    -1
@@
 F 1 "220uF" H 2985 1675 50  0000 L CNN
 F 2 "Capacitors_THT:CP_Radial_D6.3mm_P2.50mm" H 2908 1570 50  0001 C CNN
-F 3 "~" H 2870 1720 50  0001 C CNN
+F 3 "https://content.kemet.com/datasheets/KEM_A4067_A750.pdf" H 2870 1720 50  0001 C CNN
+F 4 "399-13664-ND" H 2870 1720 50  0001 C CNN "Digikey"
 	1    2870 1720
 	1    0    0    -1
@@
 F 1 "BLUE" V 3607 1683 50  0000 R CNN
 F 2 "LEDs:LED_0805" H 3660 1800 50  0001 C CNN
-F 3 "~" H 3660 1800 50  0001 C CNN
+F 3 "https://katalog.we-online.de/led/datasheet/150080BS75000.pdf" H 3660 1800 50  0001 C CNN
+F 4 "732-4982-1-ND" V 3660 1800 50  0001 C CNN "Digikey"
 	1    3660 1800
 	0    -1   -1   0
@@
 F 1 "1k" H 3728 1405 50  0000 L CNN
 F 2 "Resistors_SMD:R_0805" V 3700 1440 50  0001 C CNN
-F 3 "~" H 3660 1450 50  0001 C CNN
+F 3 "http://www.yageo.com/documents/recent/PYu-RT_1-to-0.01_RoHS_L_9.pdf" H 3660 1450 50  0001 C CNN
+F 4 "YAG1820CT-ND" H 3660 1450 50  0001 C CNN "Digikey"
 	1    3660 1450
 	1    0    0    -1
